File: wiring_diagram/ceiling.sch (KiCad schematic (older format))
At the start: 7 parts

Commit message: Adding fuel pump driver
Parts:
- F7: symbol SW_Push -> wiring_diagram-rescue:SW_Push
- SW? (x2): symbol SW_SP3T -> wiring_diagram-rescue:SW_SP3T
- U?: symbol LIN -> lin:LIN
- W, W1: symbol Lamp -> wiring_diagram-rescue:Lamp
- Z1: symbol Heater -> wiring_diagram-rescue:Heater
Connections:
- net at U?.~ (LIN): now also SW?.4
Changed lines of the file:
@@
-EESchema Schematic File Version 2
-LIBS:power
-LIBS:device
-LIBS:transistors
-LIBS:conn
-LIBS:linear
-LIBS:regul
-LIBS:74xx
-LIBS:cmos4000
-LIBS:adc-dac
-LIBS:memory
-LIBS:xilinx
-LIBS:microcontrollers
-LIBS:dsp
-LIBS:microchip
-LIBS:analog_switches
-LIBS:motorola
-LIBS:texas
-LIBS:intel
-LIBS:audio
-LIBS:interface
-LIBS:digital-audio
-LIBS:philips
-LIBS:display
-LIBS:cypress
-LIBS:siliconi
-LIBS:opto
-LIBS:atmel
-LIBS:contrib
-LIBS:valves
-LIBS:13a_switch_x4
-LIBS:switches
-LIBS:motors
-LIBS:inputs_x8
-LIBS:lin
-LIBS:sw_sp4t
-LIBS:tdc_marker_unit
+EESchema Schematic File Version 4
 LIBS:wiring_diagram-cache
-EELAYER 25 0
+EELAYER 26 0
 EELAYER END
 $Descr A4 11693 8268
@@
 $EndDescr
 $Comp
-L Lamp W
+L wiring_diagram-rescue:Lamp W
 U 1 1 5967C2A4
 P 4450 4700
@@
 $EndComp
 $Comp
-L Lamp W1
+L wiring_diagram-rescue:Lamp W1
 U 1 1 5967C2AB
 P 6800 4650
@@
 $EndComp
 $Comp
-L Heater Z1
+L wiring_diagram-rescue:Heater Z1
 U 1 1 5967CD52
 P 8850 4400
@@
 $EndComp
 $Comp
-L SW_Push F7
+L wiring_diagram-rescue:SW_Push F7
 U 1 1 5967EE1B
 P 4350 2150
@@
 $EndComp
 $Comp
-L LIN U?
+L lin:LIN U?
 U 1 1 5967EE22
 P 6000 2500
@@
 $EndComp
 $Comp
-L GND #PWR?
+L power:GND #PWR?
 U 1 1 5967EE29
 P 3950 2950
@@
 	8850 2400 8850 4250
 $Comp
-L SW_SP3T SW?
+L wiring_diagram-rescue:SW_SP3T SW?
 U 1 1 59681321
 P 3800 4700
@@
 NoConn ~ 3600 4600
 $Comp
-L SW_SP3T SW?
+L wiring_diagram-rescue:SW_SP3T SW?
 U 1 1 596817BB
 P 6250 4650
