File: wiring_diagram/floor.sch (KiCad schematic (older format))
At the start: 1 part

Commit message: Adding fuel pump driver
Parts:
- F: symbol SW_Push_Dual -> wiring_diagram-rescue:SW_Push_Dual
Changed lines of the file:
@@
-EESchema Schematic File Version 2
-LIBS:power
-LIBS:device
-LIBS:transistors
-LIBS:conn
-LIBS:linear
-LIBS:regul
-LIBS:74xx
-LIBS:cmos4000
-LIBS:adc-dac
-LIBS:memory
-LIBS:xilinx
-LIBS:microcontrollers
-LIBS:dsp
-LIBS:microchip
-LIBS:analog_switches
-LIBS:motorola
-LIBS:texas
-LIBS:intel
-LIBS:audio
-LIBS:interface
-LIBS:digital-audio
-LIBS:philips
-LIBS:display
-LIBS:cypress
-LIBS:siliconi
-LIBS:opto
-LIBS:atmel
-LIBS:contrib
-LIBS:valves
-LIBS:13a_switch_x4
-LIBS:switches
-LIBS:motors
-LIBS:inputs_x8
-LIBS:lin
-LIBS:sw_sp4t
-LIBS:tdc_marker_unit
+EESchema Schematic File Version 4
 LIBS:wiring_diagram-cache
-EELAYER 25 0
+EELAYER 26 0
 EELAYER END
 $Descr A4 11693 8268
@@
 $EndDescr
 $Comp
-L SW_Push_Dual F
+L wiring_diagram-rescue:SW_Push_Dual F
 U 1 1 59684407
 P 6100 3700
