File: wiring_diagram/lights.sch (KiCad schematic (older format))
At the start: 23 parts, among them M1 Lamp, M10 Break light, M12A Lamp, M12B Lamp, M16 Back-up light, M17 Back-up light, M2 Tail light, M3 Lamp, M4 Tail light, M5 Lamp, M6 Turn light, M7 Lamp, M8 Turn light, M9 Break light

Commit message: Adding fuel pump driver
Parts:
- L1A, L1B, L2A, L2B, M1, M10, M12A, M12B, M16, M17, M2, M3, M4, M5, M6, M7, M8, M9, X: symbol Lamp -> wiring_diagram-rescue:Lamp
- U? (x4): symbol LIN -> lin:LIN
Connections:
- net labels added: +12V, LIN
- wire segments 122 -> 147
Other:
- moved on the sheet: L2A, L2B, M3, M7, U?
