File: wiring_diagram/warning_lights.sch (KiCad schematic (older format))
At the start: 4 parts, among them K2 Alternator warning light, K3 Oil pressure warning light, K5 Turn signal warning light, K7 Break warning light

Commit message: Adding fuel pump driver
Parts:
- K2, K3, K5, K7: symbol Lamp -> wiring_diagram-rescue:Lamp
Changed lines of the file:
@@
-EESchema Schematic File Version 2
-LIBS:power
-LIBS:device
-LIBS:transistors
-LIBS:conn
-LIBS:linear
-LIBS:regul
-LIBS:74xx
-LIBS:cmos4000
-LIBS:adc-dac
-LIBS:memory
-LIBS:xilinx
-LIBS:microcontrollers
-LIBS:dsp
-LIBS:microchip
-LIBS:analog_switches
-LIBS:motorola
-LIBS:texas
-LIBS:intel
-LIBS:audio
-LIBS:interface
-LIBS:digital-audio
-LIBS:philips
-LIBS:display
-LIBS:cypress
-LIBS:siliconi
-LIBS:opto
-LIBS:atmel
-LIBS:contrib
-LIBS:valves
-LIBS:13a_switch_x4
-LIBS:switches
-LIBS:motors
-LIBS:inputs_x8
-LIBS:lin
-LIBS:sw_sp4t
-LIBS:tdc_marker_unit
+EESchema Schematic File Version 4
 LIBS:wiring_diagram-cache
-EELAYER 25 0
+EELAYER 26 0
 EELAYER END
 $Descr A4 11693 8268
@@
 $EndDescr
 $Comp
-L Lamp K7
+L wiring_diagram-rescue:Lamp K7
 U 1 1 5968CD01
 P 6250 3300
@@
 $EndComp
 $Comp
-L Lamp K3
+L wiring_diagram-rescue:Lamp K3
 U 1 1 5968CD08
 P 5100 3750
@@
 $EndComp
 $Comp
-L Lamp K2
+L wiring_diagram-rescue:Lamp K2
 U 1 1 5968CD10
 P 5350 4500
@@
 $EndComp
 $Comp
-L Lamp K5
+L wiring_diagram-rescue:Lamp K5
 U 1 1 5968D1AF
 P 6500 4050
